Commit message: Remove unused packages and upgrade to 4 Kinect cameras
- Delete mapping package entirely
- Remove pointcloud_to_grid_node and slam3d_to_grid_node (including
  pointcloud_to_grid_core.hpp, pcd2map.launch.py)
- Remove all marvelmind/fusion_gps_odom references (source, header,
  launch, CMakeLists, package.xml)
- Delete triple_concat.launch.py (no longer using astra camera)
- Upgrade from 2 Kinect cameras to 4 (front/back/right/left):
  - URDF: add camera_link + kinect1-4 links with proper orientations
  - concat.launch.py: 4-cloud concatenation from 4 kinects
  - lidar_slam_3d: expand to 4 laser scan callbacks and 4 laser clouds
  - slam_rgbd_cam.launch.py: 4 pointcloud_to_laserscan nodes covering
    full 360 degrees in 4 quadrants

https://claude.ai/code/session_0129ByhedhARqFaT83jHMq7z

File: src/robot_description/urdf/robot.xacro (robot description, xacro)
@@ -26,3 +26,134 @@
         <origin xyz="0 0 0"/>
     </joint>
+    <!-- Camera Link (center reference) -->
+    <link name="camera_link"/>
+    <joint name="base_to_camera" type="fixed">
+        <parent link="base_link"/>
+        <child link="camera_link"/>
+        <origin xyz="0.13 0 0" rpy="0 0 0"/>
+    </joint>
+    <!-- Kinect 1 - Front -->
+    <link name="kinect1_link"/>
+    <joint name="camera_to_kinect1" type="fixed">
+        <parent link="camera_link"/>
+        <child link="kinect1_link"/>
+        <origin xyz="0.15 0 0" rpy="0 0 0"/>
+    </joint>
+    <link name="kinect1_depth_frame"/>
+    <joint name="kinect1_depth_joint" type="fixed">
+        <parent link="kinect1_link"/>
+        <child link="kinect1_depth_frame"/>
+        <origin xyz="0 0 0" rpy="0 0 0"/>
+    </joint>
+    <link name="kinect1_depth_optical_frame"/>
+    <joint name="kinect1_depth_optical_joint" type="fixed">
+        <parent link="kinect1_depth_frame"/>
+        <child link="kinect1_depth_optical_frame"/>
+        <origin xyz="0 0 0" rpy="-1.5708 0 -1.5708"/>
+    </joint>
+    <link name="kinect1_rgb_frame"/>
+    <joint name="kinect1_rgb_joint" type="fixed">
+        <parent link="kinect1_link"/>
+        <child link="kinect1_rgb_frame"/>
+        <origin xyz="0 0 0" rpy="0 0 0"/>
+    </joint>
+    <link name="kinect1_rgb_optical_frame"/>
+    <joint name="kinect1_rgb_optical_joint" type="fixed">
+        <parent link="kinect1_rgb_frame"/>
+        <child link="kinect1_rgb_optical_frame"/>
+        <origin xyz="0 0 0" rpy="-1.5708 0 -1.5708"/>
+    </joint>
+    <!-- Kinect 2 - Back -->
+    <link name="kinect2_link"/>
+    <joint name="camera_to_kinect2" type="fixed">
+        <parent link="camera_link"/>
+        <child link="kinect2_link"/>
+        <origin xyz="-0.15 0 0" rpy="0 0 3.14159"/>
+    </joint>
+    <link name="kinect2_depth_frame"/>
+    <joint name="kinect2_depth_joint" type="fixed">
+        <parent link="kinect2_link"/>
+        <child link="kinect2_depth_frame"/>
+        <origin xyz="0 0 0" rpy="0 0 0"/>
+    </joint>
+    <link name="kinect2_depth_optical_frame"/>
+    <joint name="kinect2_depth_optical_joint" type="fixed">
+        <parent link="kinect2_depth_frame"/>
+        <child link="kinect2_depth_optical_frame"/>
+        <origin xyz="0 0 0" rpy="-1.5708 0 -1.5708"/>
+    </joint>
+    <link name="kinect2_rgb_frame"/>
+    <joint name="kinect2_rgb_joint" type="fixed">
+        <parent link="kinect2_link"/>
+        <child link="kinect2_rgb_frame"/>
+        <origin xyz="0 0 0" rpy="0 0 0"/>
+    </joint>
+    <link name="kinect2_rgb_optical_frame"/>
+    <joint name="kinect2_rgb_optical_joint" type="fixed">
+        <parent link="kinect2_rgb_frame"/>
+        <child link="kinect2_rgb_optical_frame"/>
+        <origin xyz="0 0 0" rpy="-1.5708 0 -1.5708"/>
+    </joint>
+    <!-- Kinect 3 - Right -->
+    <link name="kinect3_link"/>
+    <joint name="camera_to_kinect3" type="fixed">
+        <parent link="camera_link"/>
+        <child link="kinect3_link"/>
+        <origin xyz="0 -0.15 0" rpy="0 0 -1.5708"/>
+    </joint>
+    <link name="kinect3_depth_frame"/>
+    <joint name="kinect3_depth_joint" type="fixed">
+        <parent link="kinect3_link"/>
+        <child link="kinect3_depth_frame"/>
+        <origin xyz="0 0 0" rpy="0 0 0"/>
+    </joint>
+    <link name="kinect3_depth_optical_frame"/>
+    <joint name="kinect3_depth_optical_joint" type="fixed">
+        <parent link="kinect3_depth_frame"/>
+        <child link="kinect3_depth_optical_frame"/>
+        <origin xyz="0 0 0" rpy="-1.5708 0 -1.5708"/>
+    </joint>
+    <link name="kinect3_rgb_frame"/>
+    <joint name="kinect3_rgb_joint" type="fixed">
+        <parent link="kinect3_link"/>
+        <child link="kinect3_rgb_frame"/>
+        <origin xyz="0 0 0" rpy="0 0 0"/>
+    </joint>
+    <link name="kinect3_rgb_optical_frame"/>
+    <joint name="kinect3_rgb_optical_joint" type="fixed">
+        <parent link="kinect3_rgb_frame"/>
+        <child link="kinect3_rgb_optical_frame"/>
+        <origin xyz="0 0 0" rpy="-1.5708 0 -1.5708"/>
+    </joint>
+    <!-- Kinect 4 - Left -->
+    <link name="kinect4_link"/>
+    <joint name="camera_to_kinect4" type="fixed">
+        <parent link="camera_link"/>
+        <child link="kinect4_link"/>
+        <origin xyz="0 0.15 0" rpy="0 0 1.5708"/>
+    </joint>
+    <link name="kinect4_depth_frame"/>
+    <joint name="kinect4_depth_joint" type="fixed">
+        <parent link="kinect4_link"/>
+        <child link="kinect4_depth_frame"/>
+        <origin xyz="0 0 0" rpy="0 0 0"/>
+    </joint>
+    <link name="kinect4_depth_optical_frame"/>
+    <joint name="kinect4_depth_optical_joint" type="fixed">
+        <parent link="kinect4_depth_frame"/>
+        <child link="kinect4_depth_optical_frame"/>
+        <origin xyz="0 0 0" rpy="-1.5708 0 -1.5708"/>
+    </joint>
+    <link name="kinect4_rgb_frame"/>
+    <joint name="kinect4_rgb_joint" type="fixed">
+        <parent link="kinect4_link"/>
+        <child link="kinect4_rgb_frame"/>
+        <origin xyz="0 0 0" rpy="0 0 0"/>
+    </joint>
+    <link name="kinect4_rgb_optical_frame"/>
+    <joint name="kinect4_rgb_optical_joint" type="fixed">
+        <parent link="kinect4_rgb_frame"/>
+        <child link="kinect4_rgb_optical_frame"/>
+        <origin xyz="0 0 0" rpy="-1.5708 0 -1.5708"/>
+    </joint>
 </robot>
