Commit message: Fix Gazebo simulation: absolute topics, map->odom TF, RViz config
- Remove static odom link/joint from URDF (DiffDrive handles odom->base_footprint dynamically)
- Add /cmd_vel topic to DiffDrive plugin (was defaulting to /model/agv/cmd_vel)
- Make all Gazebo plugin topics absolute (/odom, /tf, /joint_states, sensor topics)
- Add map->odom static transform publisher in sim.launch.py
- Add RViz config for simulation with point cloud visualization
- Update sim_slam.launch.py to use RViz config file

https://claude.ai/code/session_0129ByhedhARqFaT83jHMq7z

File: src/robot_description/urdf/robot_sim.urdf.xacro (robot description, xacro)
@@ -162,5 +162,5 @@
         <always_on>true</always_on>
         <update_rate>${kinect_fps}</update_rate>
-        <topic>${name}/${name}/depth</topic>
+        <topic>/${name}/${name}/depth</topic>
         <gz_frame_id>${name}_depth_optical_frame</gz_frame_id>
         <camera>
@@ -180,5 +180,5 @@
         <always_on>true</always_on>
         <update_rate>${kinect_fps}</update_rate>
-        <topic>${name}/${name}/rgb</topic>
+        <topic>/${name}/${name}/rgb</topic>
         <gz_frame_id>${name}_rgb_optical_frame</gz_frame_id>
         <camera>
@@ -228,11 +228,4 @@
     <mu2>0.2</mu2>
   </gazebo>
-  <!-- Odom frame (virtual, published by diff_drive plugin) -->
-  <link name="odom"/>
-  <joint name="odom_joint" type="fixed">
-    <parent link="odom"/>
-    <child link="base_footprint"/>
-    <origin xyz="0 0 0"/>
-  </joint>
   <!-- ==================== WHEELS ========================= -->
   <xacro:drive_wheel name="left"  y_offset="${wheel_separation/2}"/>
@@ -271,6 +264,7 @@
       <max_linear_acceleration>1.0</max_linear_acceleration>
       <max_angular_acceleration>2.0</max_angular_acceleration>
-      <odom_topic>odom</odom_topic>
-      <tf_topic>tf</tf_topic>
+      <topic>/cmd_vel</topic>
+      <odom_topic>/odom</odom_topic>
+      <tf_topic>/tf</tf_topic>
       <frame_id>odom</frame_id>
       <child_frame_id>base_footprint</child_frame_id>
@@ -284,5 +278,5 @@
       <joint_name>left_wheel_joint</joint_name>
       <joint_name>right_wheel_joint</joint_name>
-      <topic>joint_states</topic>
+      <topic>/joint_states</topic>
       <update_rate>50</update_rate>
     </plugin>
